File: My-Motorola-IO.kicad_pcb (KiCad board)
At the start: 2 copper layers, 99.8 x 99.8 mm, 37 parts, among them J1 MECB_64AC, J2 PS/2_Connector, J6 Conn_02x12_Odd_Even, P1 FTDI_con, Q1 2N7000, Q2 2N7000, U1 ATF16V8, U2 RTC72421, U4 SCC2691, U5 WD65C22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

Commit message: KEYBD clk fixed, added missing pwr trace
Connections:
- U6 pad 3: KYBD_CLK -> unconnected-(U6-PB2-Pad3)
- U6 pad 4: unconnected-(U6-PB3-Pad4) -> KYBD_CLK
Routing:
- net PIA_PB3: track 123.9 -> 60.0 mm, vias 0 -> 1
- net ECB_~{WR}: track 147.2 -> 197.8 mm, vias 2 -> 0
- net ECB_~{RD}: track 199.8 -> 151.2 mm
- net +5V: track 352.2 -> 319.3 mm, vias 6 -> 0
- net /ECB_A13: track 14.7 -> 36.2 mm
- net ECB_A0: track 137.1 -> 157.0 mm, vias 0 -> 2
- net ECB_~{RESET}: track 135.0 -> 116.0 mm
- net ECB_A1: track 172.9 -> 155.7 mm
- net unconnected-(J2-Pad7): track 14.7 -> 0.00 mm
- net ECB_~{INT}: track 73.6 -> 87.3 mm
- net /ECB_D3: track 131.5 -> 142.4 mm, vias 0 -> 1
- net ECB_TxD: track 108.3 -> 119.1 mm, vias 1 -> 0
- net /ECB_A4: track 61.4 -> 53.7 mm
- net /ECB_D0: track 143.5 -> 135.9 mm, vias 0 -> 2
- net /ECB_D5: track 81.2 -> 74.5 mm, vias 1 -> 0
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Other:
- board text added: "14/10/24 - v1.4"
- board text removed: "07/06/24 - v1.3"
