File: My-Motorola-IO.kicad_sch (KiCad schematic)
At the start: 35 parts, among them J1 MECB_64AC, J2 PS/2_Connector, J6 Conn_02x12_Odd_Even, P1 FTDI_con, Q1 2N7000, U1 ATF16V8, U2 RTC72421, U4 SCC2691, U5 WD65C22, U6 ATtiny261A-P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

Commit message: updated SCC2691 reset line and battery holder
Parts:
- removed CR2032: 3.6v, TLC_Stuff:SMD CR2032, symbol dk_Battery-Holders-Clips-Contacts:BS-7
- added BT1: Battery_Cell, TLC_Stuff:SMD CR2032, symbol Device:Battery_Cell
- added Q2: 2N7000, Package_TO_SOT_THT:TO-92_Inline, symbol dk_Transistors-FETs-MOSFETs-Single:2N7000
- added R6: 1M, Resistor_THT:R_Axial_DIN0207_L6.3mm_D2.5mm_P10.16mm_Horizontal, symbol Device:R
Connections:
- net +5V: now also R6.1
- net ECB_~{RESET}: now also Q2.2 (G); no longer U4.11 (RESET)
- net GND: now also BT1.2 (-), Q2.1 (S)
- net at D2.2 (A): now also BT1.1 (+)
- new net RST: Q2.3 (D), R6.2, U4.11 (RESET)

Commit message: KEYBD clk fixed, added missing pwr trace
Connections:
- net KYBD_CLK: now also U6.4 (PB3); no longer U6.3 (PB2)
Changed lines of the file:
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@@
   (title_block
     (title "TLC SYS I/O Board for MECB")
-    (date "07/06/24")
-    (rev "1.2")
+    (date "14/10/24")
+    (rev "1.4")
     (company "TLC Stuff")
   )
@@
   (no_connect (at 31.75 86.36))
   (no_connect (at 31.75 157.48))
-  (no_connect (at 96.52 140.97))
+  (no_connect (at 96.52 138.43))
   (no_connect (at 31.75 124.46))
   (no_connect (at 31.75 66.04))
@@
     (stroke (width 0) (type default))
   )
+  (wire (pts (xy 96.52 140.97) (xy 99.06 140.97))
+    (stroke (width 0) (type default))
+  )
   (wire (pts (xy 54.61 46.99) (xy 72.39 46.99))
     (stroke (width 0) (type default))
@@
     (stroke (width 0) (type default))
   )
+  (wire (pts (xy 99.06 138.43) (xy 100.33 138.43))
+    (stroke (width 0) (type default))
+  )
   (wire (pts (xy 31.75 58.42) (xy 41.91 58.42))
     (stroke (width 0) (type default))
@@
     (stroke (width 0) (type default))
   )
-  (wire (pts (xy 96.52 138.43) (xy 100.33 138.43))
-    (stroke (width 0) (type default))
-  )
   (bus (pts (xy 54.61 172.72) (xy 54.61 182.88))
     (stroke (width 0) (type default))
@@
     (stroke (width 0) (type default))
   )
+  (wire (pts (xy 99.06 140.97) (xy 99.06 138.43))
+    (stroke (width 0) (type default))
+  )
